Commit message: Fixed visualization of upper links

File: ragnar_support/urdf/ragnar.urdf (robot description, URDF)
Before this commit: robot ragnar, 5 links, 4 joints
Links:
- added link base_link2, mass 26.5217124601092; collision mesh filename=package://ragnar_support/meshes/base_link.STL; visual mesh filename=package://ragnar_support/meshes/base_link.STL
- added link ee_link_p
- added link ee_link_r
- added link ee_link_y; collision mesh filename=package://ragnar_support/meshes/ee_link_y.STL; visual mesh filename=package://ragnar_support/meshes/ee_link_y.STL
- added link lower_arm_1_pitch
- added link lower_arm_1_yaw; collision cylinder length=0.1 radius=0.04; collision cylinder length=0.55 radius=0.02
- added link lower_arm_2_pitch
- added link lower_arm_2_yaw; collision cylinder length=0.1 radius=0.04; collision cylinder length=0.55 radius=0.02
- added link lower_arm_3_pitch
- added link lower_arm_3_yaw; collision cylinder length=0.1 radius=0.04; collision cylinder length=0.55 radius=0.02
- added link lower_arm_4_pitch
- added link lower_arm_4_yaw; collision cylinder length=0.1 radius=0.04; collision cylinder length=0.55 radius=0.02
- link base_link: mass 26.5217124601092 -> None; geometry 
- link upper_arm_1: mass 0.220403356973371 -> None; geometry collision cylinder length=0.1 radius=0.04; collision cylinder length=0.3 radius=0.02
- link upper_arm_2: mass 0.220403356973371 -> None; geometry collision cylinder length=0.1 radius=0.04; collision cylinder length=0.3 radius=0.02
- link upper_arm_3: mass 0.220403356973371 -> None; geometry collision cylinder length=0.1 radius=0.04; collision cylinder length=0.3 radius=0.02
- link upper_arm_4: mass 0.220403356973371 -> None; geometry collision cylinder length=0.1 radius=0.04; collision cylinder length=0.3 radius=0.02
Joints:
- added joint a1_j2_pitch: type revolute, parent upper_arm_1, child lower_arm_1_pitch, origin xyz=0 0.3 0 rpy=0 0 0, axis -1.0 0 0, limit lower=-3.1416 upper=3.1416 effort=0 velocity=2.618
- added joint a1_j2_yaw: type revolute, parent lower_arm_1_pitch, child lower_arm_1_yaw, origin xyz=0 0 0 rpy=0 0 0, axis 0 0 1.0, limit lower=-3.1416 upper=3.1416 effort=0 velocity=2.618
- added joint a2_j2_pitch: type revolute, parent upper_arm_2, child lower_arm_2_pitch, origin xyz=0 0.3 0 rpy=0 0 0, axis -1.0 0 0, limit lower=-3.1416 upper=3.1416 effort=0 velocity=2.618
- added joint a2_j2_yaw: type revolute, parent lower_arm_2_pitch, child lower_arm_2_yaw, origin xyz=0 0 0 rpy=0 0 0, axis 0 0 1.0, limit lower=-3.1416 upper=3.1416 effort=0 velocity=2.618
- added joint a3_j2_pitch: type revolute, parent upper_arm_3, child lower_arm_3_pitch, origin xyz=0 0.3 0 rpy=0 0 0, axis -1.0 0 0, limit lower=-3.1416 upper=3.1416 effort=0 velocity=2.618
- added joint a3_j2_yaw: type revolute, parent lower_arm_3_pitch, child lower_arm_3_yaw, origin xyz=0 0 0 rpy=0 0 0, axis 0 0 1.0, limit lower=-3.1416 upper=3.1416 effort=0 velocity=2.618
- added joint a4_j2_pitch: type revolute, parent upper_arm_4, child lower_arm_4_pitch, origin xyz=0 0.3 0 rpy=0 0 0, axis -1.0 0 0, limit lower=-3.1416 upper=3.1416 effort=0 velocity=2.618
- added joint a4_j2_yaw: type revolute, parent lower_arm_4_pitch, child lower_arm_4_yaw, origin xyz=0 0 0 rpy=0 0 0, axis 0 0 1.0, limit lower=-3.1416 upper=3.1416 effort=0 velocity=2.618
- added joint base_rotate: type fixed, parent base_link, child base_link2, origin xyz=0 0 0.05 rpy=0 0 1.57, axis 0 0 0
- added joint ee_joint_pitch: type revolute, parent ee_link_r, child ee_link_p, origin xyz=0 0 0 rpy=0 0 0, axis 1 0 0, limit lower=-3.1416 upper=3.1416 effort=0 velocity=2.618
- added joint ee_joint_roll: type revolute, parent lower_arm_1_yaw, child ee_link_r, origin xyz=0 0.550 0 rpy=0 0 0, axis 0 0 1, limit lower=-3.1416 upper=3.1416 effort=0 velocity=2.618
- added joint ee_joint_yaw: type revolute, parent ee_link_p, child ee_link_y, origin xyz=0 0 0 rpy=5.55111512312578E-17 -2.77555756156289E-17 0, axis 0 -1 0, limit lower=-3.1416 upper=3.1416 effort=0 velocity=2.618
- joint a1_j1: origin xyz=0.16 0.108 0.0576 rpy=-0.577 -0.783 -1.311 -> xyz=0.122 0.249 -0.0877 rpy=-0.577 -0.783 -1.311; parent base_link -> base_link2
- joint a2_j1: origin xyz=-0.143 0.172 -0.0087 rpy=-2.698 -0.788 -1.834 -> xyz=-0.122 0.249 -0.0877 rpy=-2.698 -0.788 -1.834; parent base_link -> base_link2
- joint a3_j1: parent base_link -> base_link2
- joint a4_j1: origin xyz=0.133 -0.211 -0.0487 rpy=-2.531 -0.788 1.307 -> xyz=0.122 -0.249 -0.0877 rpy=-2.531 -0.788 1.307; parent base_link -> base_link2

File: ragnar_support/urdf/ragnar.xacro (robot description, xacro)
@@ -1,9 +1,9 @@
 <?xml version="1.0" ?>
 <robot name="Ragnar" xmlns:xacro="http://ros.org/wiki/xacro">
-  <link name="base_link">
+  <link name="base_link"/>
+  <link name="base_link2">
     <inertial>
       <origin xyz="-4.80572213006859E-06 9.64495107789746E-06 -0.0184680705713898" rpy="0 0 0" />
-      <mass
-        value="26.5217124601092" />
+      <mass value="26.5217124601092" />
       <inertia ixx="0.936457909215975" ixy="-0.00108838510526368" ixz="1.58187182756307E-06"
         iyy="1.50216890338436" iyz="1.0107984651762E-05" izz="2.28323593907717" />
@@ -15,5 +15,5 @@
       </geometry>
       <material name="">
-        <color rgba="0.752941176470588 0.752941176470588 0.752941176470588 1" />
+        <color rgba="0.5 0.5 0.5 1" />
       </material>
     </visual>
@@ -25,4 +25,10 @@
     </collision>
   </link>
+ <joint name="base_rotate" type="fixed">
+    <origin xyz="0 0 0.05" rpy="0 0 1.57" />
+    <parent link="base_link" />
+    <child link="base_link2" />
+    <axis xyz="0 0 0" />
+  </joint>
 <xacro:include filename="$(find ragnar_support)/urdf/ragnar_upper2_macro.xacro"/>
   <xacro:ragnar_upper2 num="1" x="0.122" y="0.249" z="-0.0877" r="-0.577" p="-0.783" w="-1.311" d1="0.300" d2="0.550"/>

File: ragnar_support/urdf/ragnar_upper2_macro.xacro (robot description, xacro)
@@ -9,5 +9,5 @@
       </geometry>
       <material name="">
-        <color rgba="0.792156862745098 0.819607843137255 0.933333333333333 1" />
+        <color rgba="0.5 0.5 0.5 1" />
       </material>
     </visual>
@@ -18,5 +18,5 @@
       </geometry>
       <material name="">
-        <color rgba="0.792156862745098 0.819607843137255 0.933333333333333 1" />
+        <color rgba="0.5 0.5 0.5 1" />
       </material>
     </visual>
@@ -27,5 +27,5 @@
       </geometry>
       <material name="">
-        <color rgba="0.792156862745098 0.819607843137255 0.933333333333333 1" />
+        <color rgba="0.5 0.5 0.5 1" />
       </material>
     </collision>
@@ -36,5 +36,5 @@
       </geometry>
       <material name="">
-        <color rgba="0.792156862745098 0.819607843137255 0.933333333333333 1" />
+        <color rgba="0.5 0.5 0.5 1" />
       </material>
     </collision>
@@ -42,5 +42,5 @@
   <joint name="a${num}_j1" type="revolute">
     <origin xyz="${x} ${y} ${z}" rpy="${r} ${p} ${w}" />
-    <parent link="base_link" />
+    <parent link="base_link2" />
     <child link="upper_arm_${num}" />
     <axis xyz="-1.0 0 0" />
@@ -57,5 +57,5 @@
       </geometry>
       <material name="">
-        <color rgba="0.792156862745098 0.819607843137255 0.933333333333333 1" />
+        <color rgba="0.75 0.75 0.75 1" />
       </material>
     </visual>
@@ -66,5 +66,5 @@
       </geometry>
       <material name="">
-        <color rgba="0.792156862745098 0.819607843137255 0.933333333333333 1" />
+        <color rgba="0.75 0.75 0.75 1" />
       </material>
     </visual>
@@ -75,5 +75,5 @@
       </geometry>
       <material name="">
-        <color rgba="0.792156862745098 0.819607843137255 0.933333333333333 1" />
+        <color rgba="0.75 0.75 0.7 1" />
       </material>
     </visual>
@@ -84,5 +84,5 @@
       </geometry>
       <material name="">
-        <color rgba="0.792156862745098 0.819607843137255 0.933333333333333 1" />
+        <color rgba="0.75 0.75 0.75 1" />
       </material>
     </collision>
@@ -93,5 +93,5 @@
       </geometry>
       <material name="">
-        <color rgba="0.792156862745098 0.819607843137255 0.933333333333333 1" />
+        <color rgba="0.75 0.75 0.75 1" />
       </material>
     </collision>

Commit message: Update urdf and state publisher to show ee and base links

File: ragnar_support/urdf/ragnar.urdf (robot description, URDF)
Before this commit: robot Ragnar, 17 links, 16 joints
Links:
- link ee_link_y: geometry collision mesh filename=package://ragnar_support/meshes/ragnar_ee.STL; visual mesh filename=package://ragnar_support/meshes/ragnar_ee.STL
Joints:
- joint ee_joint_yaw: origin xyz=0 0 0 rpy=5.55111512312578E-17 -2.77555756156289E-17 0 -> xyz=0 0 0 rpy=0 0 0

File: ragnar_support/urdf/ragnar.xacro (robot description, xacro)
@@ -56,11 +56,11 @@
     <child link="ee_link_p" />
     <axis xyz="1 0 0" />
-<limit effort="0" lower="-3.1416" upper="3.1416" velocity="2.618"/>
+    <limit effort="0" lower="-3.1416" upper="3.1416" velocity="2.618"/>
   </joint>
   <link name="ee_link_y">
     <visual>
-      <origin xyz="0 0 0" rpy="0 0 0" />
+      <origin xyz="0 0 0" rpy="1.57 0 1.57" />
       <geometry>
-        <mesh filename="package://ragnar_support/meshes/ee_link_y.STL" />
+        <mesh filename="package://ragnar_support/meshes/ragnar_ee.STL" />
       </geometry>
       <material name="">
@@ -69,12 +69,12 @@
     </visual>
     <collision>
-      <origin xyz="0 0 0" rpy="0 0 0" />
+      <origin xyz="0 0 0" rpy="1.57 0 1.57" />
       <geometry>
-        <mesh filename="package://ragnar_support/meshes/ee_link_y.STL" />
+        <mesh filename="package://ragnar_support/meshes/ragnar_ee.STL" />
       </geometry>
     </collision>
   </link>
   <joint name="ee_joint_yaw" type="revolute">
-    <origin xyz="0 0 0" rpy="5.55111512312578E-17 -2.77555756156289E-17 0" />
+    <origin xyz="0 0 0" rpy="0 0 0" />
     <parent link="ee_link_p" />
     <child link="ee_link_y" />

Commit message: Fixed feedback handler and client node

File: ragnar_support/urdf/ragnar.urdf (robot description, URDF)
Before this commit: robot Ragnar, 17 links, 16 joints
Joints:
- joint a1_j1: origin xyz=0.122 0.249 -0.0877 rpy=-0.577 -0.783 -1.311 -> xyz=0.122 -0.249 -0.0877 rpy=-2.531 -0.788 1.307
- joint a2_j1: origin xyz=-0.122 0.249 -0.0877 rpy=-2.698 -0.788 -1.834 -> xyz=-0.122 -0.249 -0.0877 rpy=-0.456 -0.783 1.831
- joint a3_j1: origin xyz=-0.122 -0.249 -0.0877 rpy=-0.456 -0.783 1.831 -> xyz=-0.122 0.249 -0.0877 rpy=-2.698 -0.788 -1.834
- joint a4_j1: origin xyz=0.122 -0.249 -0.0877 rpy=-2.531 -0.788 1.307 -> xyz=0.122 0.249 -0.0877 rpy=-0.577 -0.783 -1.311
