Commit message: Changed ragnar URDF to use floating joints

File: ragnar_support/urdf/ragnar.xacro (robot description, xacro)
@@ -41,5 +41,5 @@
 <link name="ee_link_r">
   </link>
-  <joint name="ee_joint_roll" type="revolute">
+  <joint name="ee_joint_roll" type="floating">
     <origin xyz="0 0.550 0"
       rpy="0 0 0" />
@@ -51,5 +51,5 @@
   <link name="ee_link_p">
   </link>
-  <joint name="ee_joint_pitch" type="revolute">
+  <joint name="ee_joint_pitch" type="floating">
     <origin xyz="0 0 0" rpy="0 0 0" />
     <parent link="ee_link_r" />
@@ -75,5 +75,5 @@
     </collision>
   </link>
-  <joint name="ee_joint_yaw" type="revolute">
+  <joint name="ee_joint_yaw" type="floating">
     <origin xyz="0 0 0" rpy="0 0 0" />
     <parent link="ee_link_p" />

File: ragnar_support/urdf/ragnar_upper2_macro.xacro (robot description, xacro)
@@ -40,5 +40,5 @@
     </collision>
   </link>
-  <joint name="a${num}_j1" type="revolute">
+  <joint name="a${num}_j1" type="floating">
     <origin xyz="${x} ${y} ${z}" rpy="${r} ${p} ${w}" />
     <parent link="base_link2" />
@@ -97,5 +97,5 @@
     </collision>
   </link>
-  <joint name="a${num}_j2_pitch" type="revolute">
+  <joint name="a${num}_j2_pitch" type="floating">
     <origin xyz="0 ${d1} 0" rpy="0 0 0" />
     <parent link="upper_arm_${num}" />
@@ -104,5 +104,5 @@
     <limit effort="0" lower="-3.1416" upper="3.1416" velocity="2.618"/>
   </joint>
-  <joint name="a${num}_j2_yaw" type="revolute">
+  <joint name="a${num}_j2_yaw" type="floating">
     <origin xyz="0 0 0" rpy="0 0 0" />
     <parent link="lower_arm_${num}_pitch" />

Commit message: Robot now generally works w/ URDF. Requires newer version of state publisher than is in repository. Also made changes to support the ragnar_state_publisher having prefixes, but the change is not efficient.

File: ragnar_support/urdf/ragnar.xacro (robot description, xacro)
@@ -1,4 +1,11 @@
 <?xml version="1.0" ?>
 <robot name="Ragnar" xmlns:xacro="http://ros.org/wiki/xacro">
+  <xacro:include filename="$(find ragnar_support)/urdf/ragnar_upper2_macro.xacro"/>
+  <link name="world"/>
+  <joint name="world_to_ragnar" type="fixed">
+    <parent link="world"/>
+    <child link="base_link"/>
+    <origin xyz="0 0 0" />
+  </joint>
   <link name="base_link"/>
   <link name="base_link2">
@@ -25,5 +32,5 @@
     </collision>
   </link>
- <joint name="base_rotate" type="fixed">
+ <joint name="base_rotate" type="floating">
     <origin xyz="0 0 0.05" rpy="0 0 1.57" />
     <parent link="base_link" />
@@ -31,11 +38,7 @@
     <axis xyz="0 0 0" />
   </joint>
-<xacro:include filename="$(find ragnar_support)/urdf/ragnar_upper2_macro.xacro"/>
   <xacro:ragnar_upper2 num="1" x="0.122" y="0.249" z="-0.0877" r="-0.577" p="-0.783" w="-1.311" d1="0.300" d2="0.550"/>
-<xacro:include filename="$(find ragnar_support)/urdf/ragnar_upper2_macro.xacro"/>
   <xacro:ragnar_upper2 num="2" x="-0.122" y="0.249" z="-0.0877" r="-2.698" p="-0.788" w="-1.834" d1="0.300" d2="0.550"/>
-<xacro:include filename="$(find ragnar_support)/urdf/ragnar_upper2_macro.xacro"/>
   <xacro:ragnar_upper2 num="3" x="-0.122" y="-0.249" z="-0.0877" r="-0.456" p="-0.783" w="1.831" d1="0.300" d2="0.550"/>
-<xacro:include filename="$(find ragnar_support)/urdf/ragnar_upper2_macro.xacro"/>
   <xacro:ragnar_upper2 num="4" x="0.122" y="-0.249" z="-0.0877" r="-2.531" p="-0.788" w="1.307" d1="0.300" d2="0.550"/>
 <link name="ee_link_r">

Commit message: Removed extra joints and updated ragnar_state_publisher with new joint names

File: ragnar_support/urdf/ragnar.xacro (robot description, xacro)
@@ -42,24 +42,5 @@
   <xacro:ragnar_upper2 num="3" x="-0.122" y="-0.249" z="-0.0877" r="-0.456" p="-0.783" w="1.831" d1="0.300" d2="0.550"/>
   <xacro:ragnar_upper2 num="4" x="0.122" y="-0.249" z="-0.0877" r="-2.531" p="-0.788" w="1.307" d1="0.300" d2="0.550"/>
-<link name="ee_link_r">
-  </link>
-  <joint name="ee_joint_roll" type="floating">
-    <origin xyz="0 0.550 0"
-      rpy="0 0 0" />
-    <parent link="lower_arm_1_yaw" />
-    <child link="ee_link_r" />
-    <axis xyz="0 0 1" />
-    <limit effort="0" lower="-3.1416" upper="3.1416" velocity="2.618"/>
-  </joint>
-  <link name="ee_link_p">
-  </link>
-  <joint name="ee_joint_pitch" type="floating">
-    <origin xyz="0 0 0" rpy="0 0 0" />
-    <parent link="ee_link_r" />
-    <child link="ee_link_p" />
-    <axis xyz="1 0 0" />
-    <limit effort="0" lower="-3.1416" upper="3.1416" velocity="2.618"/>
-  </joint>
-  <link name="ee_link_y">
+  <link name="ee_link">
     <visual>
       <origin xyz="0 0 0" rpy="1.57 0 1.57" />
@@ -78,10 +59,8 @@
     </collision>
   </link>
-  <joint name="ee_joint_yaw" type="floating">
+  <joint name="ee_joint" type="floating">
     <origin xyz="0 0 0" rpy="0 0 0" />
-    <parent link="ee_link_p" />
-    <child link="ee_link_y" />
-    <axis xyz="0 -1 0" />
-<limit effort="0" lower="-3.1416" upper="3.1416" velocity="2.618"/>
+    <parent link="lower_arm_1" />
+    <child link="ee_link" />
   </joint>
 </robot>

File: ragnar_support/urdf/ragnar_upper2_macro.xacro (robot description, xacro)
@@ -40,5 +40,5 @@
     </collision>
   </link>
-  <joint name="a${num}_j1" type="floating">
+  <joint name="a${num}_j1" type="revolute">
     <origin xyz="${x} ${y} ${z}" rpy="${r} ${p} ${w}" />
     <parent link="base_link2" />
@@ -49,6 +49,5 @@
     <!--xacro:include filename="$(find ragnar_support)/urdf/Ragnar_lower_macro.xacro"/>
     <xacro:ragnar_lower prefix=""/-->
-  <link name="lower_arm_${num}_pitch"/>
-  <link name="lower_arm_${num}_yaw">
+  <link name="lower_arm_${num}">
     <visual>
       <origin xyz="0 0 0" rpy="0 0 0" />
@@ -97,17 +96,8 @@
     </collision>
   </link>
-  <joint name="a${num}_j2_pitch" type="floating">
+  <joint name="a${num}_j2" type="floating">
     <origin xyz="0 ${d1} 0" rpy="0 0 0" />
     <parent link="upper_arm_${num}" />
-    <child link="lower_arm_${num}_pitch" />
-    <axis xyz="-1.0 0 0" />
-    <limit effort="0" lower="-3.1416" upper="3.1416" velocity="2.618"/>
-  </joint>
-  <joint name="a${num}_j2_yaw" type="floating">
-    <origin xyz="0 0 0" rpy="0 0 0" />
-    <parent link="lower_arm_${num}_pitch" />
-    <child link="lower_arm_${num}_yaw" />
-    <axis xyz="0 0 1.0" />
-    <limit effort="0" lower="-3.1416" upper="3.1416" velocity="2.618"/>
+    <child link="lower_arm_${num}" />
   </joint>
   </xacro:macro>

Commit message: Did some minor cleanup to xacro files. Noticed that with new joint names that robot state publisher will publish transforms that do not agree with our own calculated ones. We should look at fixing this, but in the meantime I just made them floating joints

File: ragnar_support/urdf/ragnar.xacro (robot description, xacro)
@@ -1,6 +1,7 @@
 <?xml version="1.0" ?>
 <robot name="Ragnar" xmlns:xacro="http://ros.org/wiki/xacro">
-  <xacro:include filename="$(find ragnar_support)/urdf/ragnar_upper2_macro.xacro"/>
+  <xacro:include filename="$(find ragnar_support)/urdf/ragnar_macro.xacro"/>
   <link name="world"/>
+  <xacro:ragnar prefix=""/>
   <joint name="world_to_ragnar" type="fixed">
     <parent link="world"/>
@@ -8,59 +9,3 @@
     <origin xyz="0 0 0" />
   </joint>
-  <link name="base_link"/>
-  <link name="base_link2">
-    <inertial>
-      <origin xyz="-4.80572213006859E-06 9.64495107789746E-06 -0.0184680705713898" rpy="0 0 0" />
-      <mass value="26.5217124601092" />
-      <inertia ixx="0.936457909215975" ixy="-0.00108838510526368" ixz="1.58187182756307E-06"
-        iyy="1.50216890338436" iyz="1.0107984651762E-05" izz="2.28323593907717" />
-    </inertial>
-    <visual>
-      <origin xyz="0 0 0" rpy="0 0 0" />
-      <geometry>
-        <mesh filename="package://ragnar_support/meshes/base_link.STL" />
-      </geometry>
-      <material name="">
-        <color rgba="0.5 0.5 0.5 1" />
-      </material>
-    </visual>
-    <collision>
-      <origin xyz="0 0 0" rpy="0 0 0" />
-      <geometry>
-        <mesh filename="package://ragnar_support/meshes/base_link.STL" />
-      </geometry>
-    </collision>
-  </link>
- <joint name="base_rotate" type="floating">
-    <origin xyz="0 0 0.05" rpy="0 0 1.57" />
-    <parent link="base_link" />
-    <child link="base_link2" />
-    <axis xyz="0 0 0" />
-  </joint>
-  <xacro:ragnar_upper2 num="1" x="0.122" y="0.249" z="-0.0877" r="-0.577" p="-0.783" w="-1.311" d1="0.300" d2="0.550"/>
-  <xacro:ragnar_upper2 num="2" x="-0.122" y="0.249" z="-0.0877" r="-2.698" p="-0.788" w="-1.834" d1="0.300" d2="0.550"/>
-  <xacro:ragnar_upper2 num="3" x="-0.122" y="-0.249" z="-0.0877" r="-0.456" p="-0.783" w="1.831" d1="0.300" d2="0.550"/>
-  <xacro:ragnar_upper2 num="4" x="0.122" y="-0.249" z="-0.0877" r="-2.531" p="-0.788" w="1.307" d1="0.300" d2="0.550"/>
-  <link name="ee_link">
-    <visual>
-      <origin xyz="0 0 0" rpy="1.57 0 1.57" />
-      <geometry>
-        <mesh filename="package://ragnar_support/meshes/ragnar_ee.STL" />
-      </geometry>
-      <material name="">
-        <color rgba="1 0 0 1" />
-      </material>
-    </visual>
-    <collision>
-      <origin xyz="0 0 0" rpy="1.57 0 1.57" />
-      <geometry>
-        <mesh filename="package://ragnar_support/meshes/ragnar_ee.STL" />
-      </geometry>
-    </collision>
-  </link>
-  <joint name="ee_joint" type="floating">
-    <origin xyz="0 0 0" rpy="0 0 0" />
-    <parent link="lower_arm_1" />
-    <child link="ee_link" />
-  </joint>
 </robot>

File: ragnar_support/urdf/ragnar_upper2_macro.xacro (robot description, xacro)
@@ -1,6 +1,6 @@
 <?xml version="1.0" ?>
 <robot name="ragnar" xmlns:xacro="http://ros.org/wiki/xacro">
-  <xacro:macro name="ragnar_upper2" params="num x y z r p w d1 d2">
-  <link name="upper_arm_${num}">
+  <xacro:macro name="ragnar_upper2" params=" prefix num x y z r p w d1 d2">
+  <link name="${prefix}upper_arm_${num}">
     <visual>
       <origin xyz="0 0 0" rpy="0 1.57 0" />
@@ -40,8 +40,8 @@
     </collision>
   </link>
-  <joint name="a${num}_j1" type="revolute">
+  <joint name="${prefix}joint_${num}" type="floating">
     <origin xyz="${x} ${y} ${z}" rpy="${r} ${p} ${w}" />
-    <parent link="base_link2" />
-    <child link="upper_arm_${num}" />
+    <parent link="${prefix}base_link2" />
+    <child link="${prefix}upper_arm_${num}" />
     <axis xyz="-1.0 0 0" />
     <limit effort="0" lower="-3.1416" upper="3.1416" velocity="2.618"/>
@@ -49,5 +49,5 @@
     <!--xacro:include filename="$(find ragnar_support)/urdf/Ragnar_lower_macro.xacro"/>
     <xacro:ragnar_lower prefix=""/-->
-  <link name="lower_arm_${num}">
+  <link name="${prefix}lower_arm_${num}">
     <visual>
       <origin xyz="0 0 0" rpy="0 0 0" />
@@ -96,8 +96,8 @@
     </collision>
   </link>
-  <joint name="a${num}_j2" type="floating">
+  <joint name="${prefix}a${num}_j2" type="floating">
     <origin xyz="0 ${d1} 0" rpy="0 0 0" />
-    <parent link="upper_arm_${num}" />
-    <child link="lower_arm_${num}" />
+    <parent link="${prefix}upper_arm_${num}" />
+    <child link="${prefix}lower_arm_${num}" />
   </joint>
   </xacro:macro>
